Commit message: update imu

File: lab6/ex03/robot_description/urdf/depth.urdf.xacro (robot description, xacro)
@@ -12,5 +12,5 @@
     <link name="depth_frame">
         <visual>
-            <origin xyz="0.00465 -0.0475 0" rpy="${M_PI/2} 0 ${M_PI/2}"/>
+            <origin xyz="0 0 0" rpy="${M_PI/2} 0 ${M_PI/2}"/>
             <geometry>
                 <mesh filename="file://$(find robot_description)/urdf/d455.stl" scale="0.001 0.001 0.001"/>
@@ -20,5 +20,5 @@
         </visual>
         <collision>
-            <origin xyz="0.00465 -0.0475 0" rpy="${M_PI/2} 0 ${M_PI/2}"/>
+            <origin xyz="0 0 0" rpy="${M_PI/2} 0 ${M_PI/2}"/>
             <geometry>
                 <box size="0.026 0.124 0.029"/>
@@ -33,7 +33,14 @@
         </inertial>
     </link>
-    <gazebo reference="depth_frame">
+    <joint name="camera_rgb_joint" type="fixed">
+        <parent link="depth_frame"/>
+        <child link="camera_rgbd_frame"/>
+        <origin xyz="0 0 0" rpy="3.14159 3.14159 3.14159"/>
+    </joint>
+    <link name="camera_rgbd_frame"/>
+    <gazebo reference="camera_rgbd_frame">
         <sensor name='depth_sensor_frame' type='depth_camera'>"
             <gz_frame_id>robot/depth_frame</gz_frame_id>
+            <origin xyz="0 0 0" rpy="0 0 0"/>
             <pose> 0 0 0 0 0 0 </pose>
             <always_on>true</always_on>

File: lab6/ex03/robot_description/urdf/imu.urdf.xacro (robot description, xacro)
@@ -33,6 +33,7 @@
         <gravity>true</gravity>
         <sensor name='imu_sensor' type='imu'>
+            <gz_frame_id>robot/imu_sensor_link</gz_frame_id>
             <always_on>true</always_on>
-            <update_rate>1</update_rate>
+            <update_rate>50</update_rate>
             <visualize>true</visualize>
             <topic>imu</topic>
